Commit message: Fixed URDFs still looking for clearpath_robot_description package

File: urdf/a200/attachments/bumper.urdf.xacro (robot description, xacro)
@@ -6,5 +6,5 @@
             <visual>
                 <geometry>
-                    <mesh filename="package://clearpath_platform_description/meshes/a200/attachments/bumper.dae" />
+                    <mesh filename="package://clearpath_robots_sim/meshes/a200/attachments/bumper.dae" />
                 </geometry>
             </visual>

File: urdf/a200/attachments/observer_backpack.urdf.xacro (robot description, xacro)
@@ -5,5 +5,5 @@
       <visual>
         <geometry>
-          <mesh filename="package://clearpath_platform_description/meshes/a200/attachments/observer_backpack_shell.stl" />
+          <mesh filename="package://clearpath_robots_sim/meshes/a200/attachments/observer_backpack_shell.stl" />
         </geometry>
         <material name="yellow"><color rgba="0.8 0.8 0.0 1.0" /></material>
@@ -31,5 +31,5 @@
       <visual>
         <geometry>
-          <mesh filename="package://clearpath_platform_description/meshes/a200/attachments/observer_backpack_masts.stl"/>
+          <mesh filename="package://clearpath_robots_sim/meshes/a200/attachments/observer_backpack_masts.stl"/>
         </geometry>
         <material name="black"><color rgba="0.0 0.0 0.0 1.0" /></material>

File: urdf/a200/attachments/sensor_arch.urdf.xacro (robot description, xacro)
@@ -8,5 +8,5 @@
           <origin xyz="0 0 0.51" rpy="0 0 0"/>
           <geometry>
-            <mesh filename="package://clearpath_platform_description/meshes/a200/attachments/510_mm_sensor_arch.dae" />
+            <mesh filename="package://clearpath_robots_sim/meshes/a200/attachments/510_mm_sensor_arch.dae" />
           </geometry>
         </visual>
@@ -14,5 +14,5 @@
           <origin xyz="0 0 0.51" rpy="0 0 0"/>
           <geometry>
-            <mesh filename="package://clearpath_platform_description/meshes/a200/attachments/510_mm_sensor_arch.dae" />
+            <mesh filename="package://clearpath_robots_sim/meshes/a200/attachments/510_mm_sensor_arch.dae" />
           </geometry>
         </collision>
@@ -37,5 +37,5 @@
           <origin xyz="0 0 0.3" rpy="0 0 0"/>
           <geometry>
-            <mesh filename="package://clearpath_platform_description/meshes/a200/attachments/300_mm_sensor_arch.dae" />
+            <mesh filename="package://clearpath_robots_sim/meshes/a200/attachments/300_mm_sensor_arch.dae" />
           </geometry>
         </visual>
@@ -43,5 +43,5 @@
           <origin xyz="0 0 0.3" rpy="0 0 0"/>
           <geometry>
-            <mesh filename="package://clearpath_platform_description/meshes/a200/attachments/300_mm_sensor_arch.dae" />
+            <mesh filename="package://clearpath_robots_sim/meshes/a200/attachments/300_mm_sensor_arch.dae" />
           </geometry>
         </collision>

File: urdf/a200/attachments/top_plate.urdf.xacro (robot description, xacro)
@@ -9,5 +9,5 @@
             <origin xyz="0.0812 0 0" rpy="0 0 0" />
             <geometry>
-              <mesh filename="package://clearpath_platform_description/meshes/a200/attachments/large_top_plate.dae" />
+              <mesh filename="package://clearpath_robots_sim/meshes/a200/attachments/large_top_plate.dae" />
             </geometry>
           </visual>
@@ -15,5 +15,5 @@
             <origin xyz="0.0812 0 0" rpy="0 0 0"/>
             <geometry>
-              <mesh filename="package://clearpath_platform_description/meshes/a200/attachments/large_top_plate_collision.stl" />
+              <mesh filename="package://clearpath_robots_sim/meshes/a200/attachments/large_top_plate_collision.stl" />
             </geometry>
           </collision>
@@ -54,5 +54,5 @@
             <origin xyz="0.272 0 0.019"/>
             <geometry>
-              <mesh filename="package://clearpath_platform_description/meshes/a200/attachments/user_rail.dae" />
+              <mesh filename="package://clearpath_robots_sim/meshes/a200/attachments/user_rail.dae" />
             </geometry>
           </visual>
@@ -69,5 +69,5 @@
             <origin xyz="0.0812 0 0" rpy="0 0 0" />
             <geometry>
-              <mesh filename="package://clearpath_platform_description/meshes/a200/attachments/top_plate.dae" />
+              <mesh filename="package://clearpath_robots_sim/meshes/a200/attachments/top_plate.dae" />
             </geometry>
           </visual>
@@ -75,5 +75,5 @@
             <origin xyz="0.0812 0 0" rpy="0 0 0"/>
             <geometry>
-              <mesh filename="package://clearpath_platform_description/meshes/a200/attachments/top_plate.stl" />
+              <mesh filename="package://clearpath_robots_sim/meshes/a200/attachments/top_plate.stl" />
             </geometry>
           </collision>
@@ -116,5 +116,5 @@
             <material name="clearpath_dark_grey" />
             <geometry>
-              <mesh filename="package://clearpath_platform_description/meshes/a200/attachments/pacs_top_plate.stl" />
+              <mesh filename="package://clearpath_robots_sim/meshes/a200/attachments/pacs_top_plate.stl" />
             </geometry>
           </visual>

File: urdf/a200/wheels/wheel.urdf.xacro (robot description, xacro)
@@ -11,5 +11,5 @@
         <origin xyz="0 0 0" rpy="0 0 0" />
         <geometry>
-          <mesh filename="package://clearpath_platform_description/meshes/a200/wheel.dae" />
+          <mesh filename="package://clearpath_robots_sim/meshes/a200/wheel.dae" />
         </geometry>
       </visual>

File: urdf/a300/a300.urdf.xacro (robot description, xacro)
@@ -28,15 +28,15 @@
       <visual>
         <geometry>
-          <mesh filename="package://clearpath_platform_description/meshes/a300/chassis.dae" />
+          <mesh filename="package://clearpath_robots_sim/meshes/a300/chassis.dae" />
         </geometry>
       </visual>
       <visual>
         <geometry>
-          <mesh filename="package://clearpath_platform_description/meshes/a300/livery.dae" />
+          <mesh filename="package://clearpath_robots_sim/meshes/a300/livery.dae" />
         </geometry>
       </visual>
       <visual>
         <geometry>
-          <mesh filename="package://clearpath_platform_description/meshes/a300/status_lights.dae" />
+          <mesh filename="package://clearpath_robots_sim/meshes/a300/status_lights.dae" />
         </geometry>
       </visual>
@@ -44,5 +44,5 @@
         <material name="clearpath_yellow"/>
         <geometry>
-          <mesh filename="package://clearpath_platform_description/meshes/a300/chassis_collision.stl" />
+          <mesh filename="package://clearpath_robots_sim/meshes/a300/chassis_collision.stl" />
         </geometry>
       </collision>

File: urdf/a300/attachments/bumper.urdf.xacro (robot description, xacro)
@@ -7,5 +7,5 @@
         <origin xyz="-0.368500 0 -0.018050"/>
         <geometry>
-          <mesh filename="package://clearpath_platform_description/meshes/a300/attachments/bumper.dae" />
+          <mesh filename="package://clearpath_robots_sim/meshes/a300/attachments/bumper.dae" />
         </geometry>
       </visual>
@@ -13,5 +13,5 @@
         <origin xyz="-0.368500 0 -0.018050"/>
         <geometry>
-          <mesh filename="package://clearpath_platform_description/meshes/a300/attachments/bumper_collision.stl" />
+          <mesh filename="package://clearpath_robots_sim/meshes/a300/attachments/bumper_collision.stl" />
         </geometry>
       </collision>

File: urdf/a300/attachments/top_plate.urdf.xacro (robot description, xacro)
@@ -13,5 +13,5 @@
             <origin xyz="0.0 0.0 ${-offset_z}"/>
             <geometry>
-              <mesh filename="package://clearpath_platform_description/meshes/a300/attachments/top_plate.dae" />
+              <mesh filename="package://clearpath_robots_sim/meshes/a300/attachments/top_plate.dae" />
             </geometry>
           </visual>

File: urdf/a300/mobility/diff_drive.urdf.xacro (robot description, xacro)
@@ -30,10 +30,10 @@
       <visual>
         <geometry>
-          <mesh filename="package://clearpath_platform_description/meshes/a300/mobility/diff_drive.dae" />
+          <mesh filename="package://clearpath_robots_sim/meshes/a300/mobility/diff_drive.dae" />
         </geometry>
       </visual>
       <collision>
         <geometry>
-          <mesh filename="package://clearpath_platform_description/meshes/a300/mobility/diff_drive_collision.stl" />
+          <mesh filename="package://clearpath_robots_sim/meshes/a300/mobility/diff_drive_collision.stl" />
         </geometry>
       </collision>

File: urdf/a300/wheels/wheel.urdf.xacro (robot description, xacro)
@@ -15,5 +15,5 @@
         <material name="clearpath_dark_grey"/>
         <geometry>
-          <mesh filename="package://clearpath_platform_description/meshes/a300/mobility/${wheel_mesh}" />
+          <mesh filename="package://clearpath_robots_sim/meshes/a300/mobility/${wheel_mesh}" />
         </geometry>
       </visual>

File: urdf/dd100/attachments/top_plate.urdf.xacro (robot description, xacro)
@@ -18,5 +18,5 @@
           <material name="clearpath_dark_grey" />
           <geometry>
-            <mesh filename="package://clearpath_platform_description/meshes/dd100/attachments/pacs_top_plate.stl" />
+            <mesh filename="package://clearpath_robots_sim/meshes/dd100/attachments/pacs_top_plate.stl" />
           </geometry>
         </visual>

File: urdf/dd100/dd100.urdf.xacro (robot description, xacro)
@@ -29,5 +29,5 @@
         <origin xyz="0 0 0" rpy="0 0 0"/>
         <geometry>
-          <mesh filename="package://clearpath_platform_description/meshes/dd100/chassis.dae"/>
+          <mesh filename="package://clearpath_robots_sim/meshes/dd100/chassis.dae"/>
         </geometry>
       </visual>
@@ -35,5 +35,5 @@
         <origin xyz="0 0 0"/>
         <geometry>
-          <mesh filename="package://clearpath_platform_description/meshes/dd100/chassis_collision.stl"/>
+          <mesh filename="package://clearpath_robots_sim/meshes/dd100/chassis_collision.stl"/>
         </geometry>
       </collision>

File: urdf/dd100/wheels/wheel.urdf.xacro (robot description, xacro)
@@ -6,5 +6,5 @@
         <origin xyz="0 0 0" rpy="0 0 0"/>
         <geometry>
-          <mesh filename="package://clearpath_platform_description/meshes/dd100/wheel.stl"/>
+          <mesh filename="package://clearpath_robots_sim/meshes/dd100/wheel.stl"/>
         </geometry>
         <material name="clearpath_black" />

File: urdf/dd150/dd150.urdf.xacro (robot description, xacro)
@@ -29,5 +29,5 @@
         <origin xyz="0 0 0" rpy="0 0 0"/>
         <geometry>
-          <mesh filename="package://clearpath_platform_description/meshes/dd100/chassis.dae"/>
+          <mesh filename="package://clearpath_robots_sim/meshes/dd100/chassis.dae"/>
         </geometry>
       </visual>
@@ -35,5 +35,5 @@
         <origin xyz="0 0 0"/>
         <geometry>
-          <mesh filename="package://clearpath_platform_description/meshes/dd100/chassis_collision.stl"/>
+          <mesh filename="package://clearpath_robots_sim/meshes/dd100/chassis_collision.stl"/>
         </geometry>
       </collision>

File: urdf/dd150/wheels/wheel.urdf.xacro (robot description, xacro)
@@ -6,5 +6,5 @@
         <origin xyz="0 0 0" rpy="0 0 0"/>
         <geometry>
-          <mesh filename="package://clearpath_platform_description/meshes/dd100/wheel.stl"/>
+          <mesh filename="package://clearpath_robots_sim/meshes/dd100/wheel.stl"/>
         </geometry>
         <material name="clearpath_black" />

File: urdf/do100/do100.urdf.xacro (robot description, xacro)
@@ -28,5 +28,5 @@
         <origin xyz="0 0 0" rpy="0 0 0"/>
         <geometry>
-          <mesh filename="package://clearpath_platform_description/meshes/do100/omni_chassis.dae"/>
+          <mesh filename="package://clearpath_robots_sim/meshes/do100/omni_chassis.dae"/>
         </geometry>
       </visual>
@@ -34,5 +34,5 @@
         <origin xyz="0 0 0"/>
         <geometry>
-          <mesh filename="package://clearpath_platform_description/meshes/do100/omni_chassis_collision.stl"/>
+          <mesh filename="package://clearpath_robots_sim/meshes/do100/omni_chassis_collision.stl"/>
         </geometry>
       </collision>

File: urdf/do100/wheels/wheel.urdf.xacro (robot description, xacro)
@@ -6,5 +6,5 @@
         <origin xyz="0 ${side * 0.027} 0" rpy="0 0 ${PI/2}"/>
         <geometry>
-          <mesh filename="package://clearpath_platform_description/meshes/do100/mecanum_wheel.dae" scale="${side} 1 1" />
+          <mesh filename="package://clearpath_robots_sim/meshes/do100/mecanum_wheel.dae" scale="${side} 1 1" />
         </geometry>
       </visual>

File: urdf/j100/attachments/fender.urdf.xacro (robot description, xacro)
@@ -7,8 +7,8 @@
         <geometry>
           <xacro:if value="${model == 'default'}">
-            <mesh filename="package://clearpath_platform_description/meshes/j100/attachments/default_fender.stl" />
+            <mesh filename="package://clearpath_robots_sim/meshes/j100/attachments/default_fender.stl" />
           </xacro:if>
           <xacro:if value="${model == 'sensor'}">
-            <mesh filename="package://clearpath_platform_description/meshes/j100/attachments/sensor_fender.stl" />
+            <mesh filename="package://clearpath_robots_sim/meshes/j100/attachments/sensor_fender.stl" />
           </xacro:if>
         </geometry>

File: urdf/j100/attachments/top_plate.urdf.xacro (robot description, xacro)
@@ -7,5 +7,5 @@
             <origin xyz="0 0 0" rpy="0 0 0"/>
             <geometry>
-              <mesh filename="package://clearpath_platform_description/meshes/j100/attachments/ark_enclosure.stl"/>
+              <mesh filename="package://clearpath_robots_sim/meshes/j100/attachments/ark_enclosure.stl"/>
             </geometry>
             <material name="clearpath_dark_grey" />

File: urdf/j100/j100.urdf.xacro (robot description, xacro)
@@ -71,5 +71,5 @@
         <origin xyz="0 0 ${footprint_vertical_offset}" rpy="${PI/2} 0 ${PI/2}"/>
         <geometry>
-          <mesh filename="package://clearpath_platform_description/meshes/j100/j100_base.stl"/>
+          <mesh filename="package://clearpath_robots_sim/meshes/j100/j100_base.stl"/>
         </geometry>
         <material name="clearpath_dark_grey" />
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